File: schema/decoder.sch (KiCad schematic (older format))
At the start: 17 parts, among them Q1 2N2905, U1 7402, U2 HEF4526B, U3 TLC555

Commit message: led driver MOS, correct opamp
Other:
- note added: "Missing pulse detector"
Changed lines of the file:
@@
 Connection ~ 4950 1800
 Wire Wire Line
-	4950 1650 4950 2100
+	4950 1650 4950 1800
+Wire Wire Line
+	4950 1800 4950 1950
+Wire Wire Line
+	4950 1950 4950 2100
 Connection ~ 4400 2100
 Wire Wire Line
@@
 	4650 1950 4300 1950
 Wire Wire Line
-	4400 1550 4400 3200
+	4400 1550 4400 2100
 Wire Wire Line
-	4300 1550 4300 3200
+	4400 2100 4400 3200
+Wire Wire Line
+	4300 1550 4300 1950
+Wire Wire Line
+	4300 1950 4300 3200
 Connection ~ 4200 1800
 Wire Wire Line
@@
 	4650 1650 4100 1650
 Wire Wire Line
-	4100 950  4400 950
+	4100 950  4200 950
+Wire Wire Line
+	4200 950  4250 950
+Wire Wire Line
+	4250 950  4300 950
+Wire Wire Line
+	4300 950  4400 950
 Connection ~ 4250 950
 Wire Wire Line
@@
 	3900 5800 3900 5950
 Wire Wire Line
-	3800 5800 4050 5800
+	3800 5800 3900 5800
+Wire Wire Line
+	3900 5800 4050 5800
 Wire Wire Line
 	4350 5800 4500 5800
@@
 Connection ~ 8300 3850
 Wire Wire Line
-	8300 5700 5700 5700
+	8300 5700 5800 5700
 Wire Wire Line
-	8300 3650 8300 5950
+	5800 5700 5700 5700
+Wire Wire Line
+	8300 3650 8300 3850
+Wire Wire Line
+	8300 3850 8300 5700
+Wire Wire Line
+	8300 5700 8300 5950
 Wire Wire Line
 	7850 3850 8300 3850
@@
 Connection ~ 6800 5050
 Wire Wire Line
-	6800 5000 6800 5150
+	6800 5000 6800 5050
+Wire Wire Line
+	6800 5050 6800 5150
 Wire Wire Line
 	7000 5050 6800 5050
@@
 	6800 3950 6850 3950
 Wire Wire Line
-	6800 3450 6800 4600
+	6800 3450 6800 3650
+Wire Wire Line
+	6800 3650 6800 3950
+Wire Wire Line
+	6800 3950 6800 4550
+Wire Wire Line
+	6800 4550 6800 4600
 Wire Wire Line
 	3350 3750 3350 2900
@@
 Connection ~ 6400 3850
 Wire Wire Line
-	3000 2900 6400 2900
+	1650 2900 3350 2900
+Wire Wire Line
+	3350 2900 6400 2900
 Wire Wire Line
 	7350 4150 7350 4250
@@
 	6400 4800 6500 4800
 Wire Wire Line
-	6400 2900 6400 4800
+	6400 2900 6400 3850
+Wire Wire Line
+	6400 3850 6400 4800
 Wire Wire Line
 	6850 3850 6400 3850
@@
 	3950 4350 3250 4350
 Wire Wire Line
-	3250 4000 3250 4500
+	3250 4000 3250 4350
+Wire Wire Line
+	3250 4350 3250 4500
 Wire Wire Line
 	3450 4000 3250 4000
@@
 	3150 4100 3450 4100
 Wire Wire Line
-	3150 3550 3150 4100
+	3150 3550 3150 3650
+Wire Wire Line
+	3150 3650 3150 4100
 Wire Wire Line
 	3450 3650 3150 3650
@@
 Connection ~ 4200 950
 Wire Wire Line
-	4200 1550 4200 3200
+	4200 1550 4200 1800
 Wire Wire Line
-	4100 1550 4100 3200
+	4200 1800 4200 3200
 Wire Wire Line
-	2050 5700 2250 5700
+	4100 1550 4100 1650
+Wire Wire Line
+	4100 1650 4100 3200
+Wire Wire Line
+	2050 5700 2150 5700
+Wire Wire Line
+	2150 5700 2250 5700
 Wire Wire Line
 	2050 5700 2050 2700
@@
 Text HLabel 9950 6050 2    60   Output ~ 0
 OUTPUT
-Text HLabel 3000 2900 0    60   Input ~ 0
+Text HLabel 1650 2900 0    60   Input ~ 0
 DECODER_INPUT
+Wire Notes Line
+	6200 1900 6200 5400
+Wire Notes Line
+	6200 5400 8800 5400
+Wire Notes Line
+	8800 1900 6200 1900
+Text Notes 6250 2100 0    100  ~ 0
+Missing pulse detector
+Wire Notes Line
+	8800 5400 8800 1900
 $EndSCHEMATC

Commit message: decoder documentation
Other:
- note added: "Counter & comparator"
- note added: "compare match"
- note added: "counter reset"
- note added: "missing pulse (end of burst)"
- moved on the sheet: C3, C4, Q1, R7, R8, U3

Commit message: LED driver doc
Other:
- note added: "Counter"
- note added: "terminal count"
- note removed: "Counter & comparator"
- note removed: "compare match"
Changed lines of the file:
@@
 L GND #PWR3
 U 1 1 58C0583B
-P 3250 4500
-F 0 "#PWR3" H 3250 4250 50  0001 C CNN
-F 1 "GND" H 3250 4350 50  0000 C CNN
-F 2 "" H 3250 4500 50  0000 C CNN
-F 3 "" H 3250 4500 50  0000 C CNN
-	1    3250 4500
+P 3350 4500
+F 0 "#PWR3" H 3350 4250 50  0001 C CNN
+F 1 "GND" H 3350 4350 50  0000 C CNN
+F 2 "" H 3350 4500 50  0000 C CNN
+F 3 "" H 3350 4500 50  0000 C CNN
+	1    3350 4500
 	1    0    0    -1
 $EndComp
@@
 Text Notes 6550 1150 0    100  ~ 0
 Missing pulse detector
-Text Notes 3700 4750 0    100  ~ 0
-Counter & comparator
+Text Notes 2550 800  0    100  ~ 0
+Counter
 Wire Wire Line
 	2550 5700 2600 5700
@@
 Wire Wire Line
 	4650 4100 6200 4100
-Connection ~ 3250 4350
-Wire Wire Line
-	3950 4350 3250 4350
-Wire Wire Line
-	3250 4000 3250 4350
-Wire Wire Line
-	3250 4350 3250 4500
-Wire Wire Line
-	3450 4000 3250 4000
+Connection ~ 3350 4350
+Wire Wire Line
+	3950 4350 3350 4350
+Wire Wire Line
+	3350 4000 3350 4350
+Wire Wire Line
+	3350 4350 3350 4500
+Wire Wire Line
+	3450 4000 3350 4000
 Connection ~ 3150 3650
 Wire Wire Line
@@
 Text Notes 3000 2650 0    60   ~ 0
 counter reset
-Text Notes 6250 6000 0    60   ~ 0
-compare match
 Text Notes 7250 5300 0    60   ~ 0
 missing pulse (end of burst)
+Text Notes 4900 4050 0    60   ~ 0
+terminal count
 $EndSCHEMATC

Commit message: fix values of decoder for 1ms period
Parts:
- C1: value 1nF -> 100nF
- C2, C3: value 10nF -> 100nF
- R1, R2: value 4.5k -> 10k
Connections:
- net at R8.2, U1.12, U3.3 (OUT): now also R1.2; no longer U1.2, U1.5
- net at C1.1, R1.1: now also U1.2, U1.5; no longer U2.3 (PL)
- net at U1.3: now also U2.3 (PL); no longer R1.2
Other:
- note added: "counter reset\n(active high)"
- note added: "falling edge detector"
- note added: "missing pulse (end of burst)\nactive low"
- note added: "reset delay"
- note removed: "counter reset"
- note removed: "missing pulse (end of burst)"
- moved on the sheet: C1, C2, R1, R2, U1A, U1B
Changed lines of the file:
@@
 P 7300 3850
 F 0 "C3" H 7325 3950 50  0000 L CNN
-F 1 "10nF" H 7325 3750 50  0000 L CNN
+F 1 "100nF" H 7325 3750 50  0000 L CNN
 F 2 "" H 7338 3700 50  0000 C CNN
 F 3 "" H 7300 3850 50  0000 C CNN
@@
 $Comp
 L 7402 U1
-U 1 1 58C07DEF
-P 3200 5700
-F 0 "U1" H 3200 5750 50  0000 C CNN
-F 1 "7402" H 3250 5650 50  0000 C CNN
-F 2 "" H 3200 5700 50  0000 C CNN
-F 3 "" H 3200 5700 50  0000 C CNN
-	1    3200 5700
-	-1   0    0    1
-$EndComp
-$Comp
-L 7402 U1
 U 2 1 58C07EDD
-P 5100 5800
-F 0 "U1" H 5100 5850 50  0000 C CNN
-F 1 "7402" H 5150 5750 50  0000 C CNN
-F 2 "" H 5100 5800 50  0000 C CNN
-F 3 "" H 5100 5800 50  0000 C CNN
-	2    5100 5800
+P 4700 5800
+F 0 "U1" H 4700 5850 50  0000 C CNN
+F 1 "7402" H 4750 5750 50  0000 C CNN
+F 2 "" H 4700 5800 50  0000 C CNN
+F 3 "" H 4700 5800 50  0000 C CNN
+	2    4700 5800
 	-1   0    0    1
 $EndComp
@@
 L GND #PWR8
 U 1 1 58C07F5B
-P 5800 6000
-F 0 "#PWR8" H 5800 5750 50  0001 C CNN
-F 1 "GND" H 5800 5850 50  0000 C CNN
-F 2 "" H 5800 6000 50  0000 C CNN
-F 3 "" H 5800 6000 50  0000 C CNN
-	1    5800 6000
+P 5400 6000
+F 0 "#PWR8" H 5400 5750 50  0001 C CNN
+F 1 "GND" H 5400 5850 50  0000 C CNN
+F 2 "" H 5400 6000 50  0000 C CNN
+F 3 "" H 5400 6000 50  0000 C CNN
+	1    5400 6000
 	1    0    0    -1
 $EndComp
@@
 L R R2
 U 1 1 58C080F8
-P 4200 5800
-F 0 "R2" V 4280 5800 50  0000 C CNN
-F 1 "4.5k" V 4200 5800 50  0000 C CNN
-F 2 "" V 4130 5800 50  0000 C CNN
-F 3 "" H 4200 5800 50  0000 C CNN
-	1    4200 5800
+P 3800 5800
+F 0 "R2" V 3880 5800 50  0000 C CNN
+F 1 "10k" V 3800 5800 50  0000 C CNN
+F 2 "" V 3730 5800 50  0000 C CNN
+F 3 "" H 3800 5800 50  0000 C CNN
+	1    3800 5800
 	0    1    1    0
 $EndComp
@@
 L C C2
 U 1 1 58C08727
-P 3900 6100
-F 0 "C2" H 3925 6200 50  0000 L CNN
-F 1 "10nF" H 3925 6000 50  0000 L CNN
-F 2 "" H 3938 5950 50  0000 C CNN
-F 3 "" H 3900 6100 50  0000 C CNN
-	1    3900 6100
+P 3500 6100
+F 0 "C2" H 3525 6200 50  0000 L CNN
+F 1 "100nF" H 3525 6000 50  0000 L CNN
+F 2 "" H 3538 5950 50  0000 C CNN
+F 3 "" H 3500 6100 50  0000 C CNN
+	1    3500 6100
 	1    0    0    -1
 $EndComp
@@
 L GND #PWR5
 U 1 1 58C08807
-P 3900 6250
-F 0 "#PWR5" H 3900 6000 50  0001 C CNN
-F 1 "GND" H 3900 6100 50  0000 C CNN
-F 2 "" H 3900 6250 50  0000 C CNN
-F 3 "" H 3900 6250 50  0000 C CNN
-	1    3900 6250
+P 3500 6250
+F 0 "#PWR5" H 3500 6000 50  0001 C CNN
+F 1 "GND" H 3500 6100 50  0000 C CNN
+F 2 "" H 3500 6250 50  0000 C CNN
+F 3 "" H 3500 6250 50  0000 C CNN
+	1    3500 6250
 	1    0    0    -1
 $EndComp
@@
 L R R1
 U 1 1 58C089F9
-P 2400 5700
-F 0 "R1" V 2480 5700 50  0000 C CNN
-F 1 "4.5k" V 2400 5700 50  0000 C CNN
-F 2 "" V 2330 5700 50  0000 C CNN
-F 3 "" H 2400 5700 50  0000 C CNN
-	1    2400 5700
+P 5850 5350
+F 0 "R1" V 5930 5350 50  0000 C CNN
+F 1 "10k" V 5850 5350 50  0000 C CNN
+F 2 "" V 5780 5350 50  0000 C CNN
+F 3 "" H 5850 5350 50  0000 C CNN
+	1    5850 5350
 	0    -1   -1   0
 $EndComp
@@
 L C C1
 U 1 1 58C08CC1
-P 2150 5950
-F 0 "C1" H 2175 6050 50  0000 L CNN
-F 1 "1nF" H 2175 5850 50  0000 L CNN
-F 2 "" H 2188 5800 50  0000 C CNN
-F 3 "" H 2150 5950 50  0000 C CNN
-	1    2150 5950
+P 5550 5500
+F 0 "C1" H 5575 5600 50  0000 L CNN
+F 1 "100nF" H 5575 5400 50  0000 L CNN
+F 2 "" H 5588 5350 50  0000 C CNN
+F 3 "" H 5550 5500 50  0000 C CNN
+	1    5550 5500
 	1    0    0    -1
 $EndComp
@@
 L GND #PWR1
 U 1 1 58C08D75
-P 2150 6100
-F 0 "#PWR1" H 2150 5850 50  0001 C CNN
-F 1 "GND" H 2150 5950 50  0000 C CNN
-F 2 "" H 2150 6100 50  0000 C CNN
-F 3 "" H 2150 6100 50  0000 C CNN
-	1    2150 6100
+P 5550 5650
+F 0 "#PWR1" H 5550 5400 50  0001 C CNN
+F 1 "GND" H 5550 5500 50  0000 C CNN
+F 2 "" H 5550 5650 50  0000 C CNN
+F 3 "" H 5550 5650 50  0000 C CNN
+	1    5550 5650
 	1    0    0    -1
 $EndComp
@@
 Counter
 Wire Wire Line
-	2550 5700 2600 5700
-Wire Wire Line
 	4250 950  4250 800
 Wire Wire Line
@@
 Connection ~ 4950 1800
 Wire Wire Line
-	4950 1650 4950 1800
-Wire Wire Line
-	4950 1800 4950 1950
-Wire Wire Line
-	4950 1950 4950 2100
+	4950 1650 4950 2100
 Connection ~ 4400 2100
 Wire Wire Line
@@
 	4650 1950 4300 1950
 Wire Wire Line
-	4400 1550 4400 2100
-Wire Wire Line
-	4400 2100 4400 3200
-Wire Wire Line
-	4300 1550 4300 1950
-Wire Wire Line
-	4300 1950 4300 3200
+	4400 1550 4400 3200
+Wire Wire Line
+	4300 1550 4300 3200
 Connection ~ 4200 1800
 Wire Wire Line
@@
 	4650 1650 4100 1650
 Wire Wire Line
-	4100 950  4200 950
-Wire Wire Line
-	4200 950  4250 950
-Wire Wire Line
-	4250 950  4300 950
-Wire Wire Line
-	4300 950  4400 950
+	4100 950  4400 950
 Connection ~ 4250 950
 Wire Wire Line
 	3750 3100 3750 3200
 Wire Wire Line
-	2150 6100 2150 6100
-Wire Wire Line
-	8600 5350 5700 5350
-Wire Wire Line
-	5700 5350 3800 5350
-Wire Wire Line
-	3800 5350 3800 5600
-Connection ~ 3900 5800
-Wire Wire Line
-	3900 5800 3900 5950
-Wire Wire Line
-	3800 5800 3900 5800
-Wire Wire Line
-	3900 5800 4050 5800
-Wire Wire Line
-	4350 5800 4500 5800
-Wire Wire Line
-	5800 5900 5700 5900
-Wire Wire Line
-	5800 6000 5800 5900
+	5550 5650 5550 5650
+Wire Wire Line
+	3400 5350 5700 5350
+Wire Wire Line
+	3400 5350 3400 5600
+Connection ~ 3500 5800
+Wire Wire Line
+	3500 5800 3500 5950
+Wire Wire Line
+	3400 5800 3650 5800
+Wire Wire Line
+	3950 5800 4100 5800
+Wire Wire Line
+	5400 5900 5300 5900
+Wire Wire Line
+	5400 6000 5400 5900
 Wire Wire Line
 	9800 6050 9950 6050
@@
 Connection ~ 8600 2900
 Wire Wire Line
-	8600 2700 8600 2900
-Wire Wire Line
-	8600 2900 8600 5350
-Wire Wire Line
-	8600 5350 8600 5950
+	8600 2700 8600 5950
 Wire Wire Line
 	8150 2900 8600 2900
@@
 Connection ~ 7100 4100
 Wire Wire Line
-	7100 4050 7100 4100
-Wire Wire Line
-	7100 4100 7100 4200
+	7100 4050 7100 4200
 Wire Wire Line
 	7300 4100 7100 4100
@@
 	7100 3000 7150 3000
 Wire Wire Line
-	7100 2500 7100 2700
-Wire Wire Line
-	7100 2700 7100 3000
-Wire Wire Line
-	7100 3000 7100 3600
-Wire Wire Line
-	7100 3600 7100 3650
+	7100 2500 7100 3650
 Wire Wire Line
 	3350 3750 3350 2900
@@
 	6700 3850 6800 3850
 Wire Wire Line
-	1650 2900 3350 2900
-Wire Wire Line
-	3350 2900 6700 2900
-Wire Wire Line
-	6700 2900 7150 2900
+	1650 2900 7150 2900
 Wire Wire Line
 	6700 2900 6700 3850
@@
 	3950 4350 3350 4350
 Wire Wire Line
-	3350 4000 3350 4350
-Wire Wire Line
-	3350 4350 3350 4500
+	3350 4000 3350 4500
 Wire Wire Line
 	3450 4000 3350 4000
@@
 	3150 4100 3450 4100
 Wire Wire Line
-	3150 3550 3150 3650
-Wire Wire Line
-	3150 3650 3150 4100
+	3150 3550 3150 4100
 Wire Wire Line
 	3450 3650 3150 3650
@@
 Connection ~ 4200 950
 Wire Wire Line
-	4200 1550 4200 1800
-Wire Wire Line
-	4200 1800 4200 3200
-Wire Wire Line
-	4100 1550 4100 1650
-Wire Wire Line
-	4100 1650 4100 3200
-Wire Wire Line
-	2050 5700 2150 5700
-Wire Wire Line
-	2150 5700 2250 5700
+	4200 1550 4200 3200
+Wire Wire Line
+	4100 1550 4100 3200
 Wire Wire Line
 	2050 5700 2050 2700
-Wire Wire Line
-	2150 5800 2150 5700
-Connection ~ 2150 5700
 Wire Notes Line
 	6500 950  6500 4450
@@
 Connection ~ 8600 5350
 Wire Wire Line
-	5700 5700 5700 5350
-Connection ~ 5700 5350
+	5300 5700 5300 5350
+Connection ~ 5300 5350
 Text Notes 3000 2650 0    60   ~ 0
-counter reset
+counter reset\n(active high)
 Text Notes 7250 5300 0    60   ~ 0
-missing pulse (end of burst)
+missing pulse (end of burst)\nactive low
 Text Notes 4900 4050 0    60   ~ 0
 terminal count
+Text Notes 3550 6700 0    60   ~ 0
+falling edge detector
+$Comp
+L 7402 U1
+U 1 1 58C07DEF
+P 2800 5700
+F 0 "U1" H 2800 5750 50  0000 C CNN
+F 1 "7402" H 2850 5650 50  0000 C CNN
+F 2 "" H 2800 5700 50  0000 C CNN
+F 3 "" H 2800 5700 50  0000 C CNN
+	1    2800 5700
+	-1   0    0    1
+$EndComp
+Wire Wire Line
+	2050 5700 2200 5700
+Connection ~ 5550 5350
+Wire Wire Line
+	6000 5350 8600 5350
+Text Notes 5450 5150 0    60   ~ 0
+reset delay
 $EndSCHEMATC

Commit message: correct led driver name
Parts:
- Q1: value 2N2905 -> BC177
Changed lines of the file:
@@
 P 7000 3850
 F 0 "Q1" H 7000 4000 50  0000 R CNN
-F 1 "2N2905" H 7050 3700 50  0000 R CNN
+F 1 "BC177" H 7050 3700 50  0000 R CNN
 F 2 "" H 7200 3950 50  0000 C CNN
 F 3 "" H 7000 3850 50  0000 C CNN

Commit message: NOR update
Connections:
- net GND: now also U1.2, U1.8; no longer U1.6, U1.9
- net OUTPUT: now also U1.4; no longer U1.11
- net at R1.2, R8.2, U3.3 (OUT): now also U1.6; no longer U1.12
- net at U2.12 (TC): now also U1.1; no longer U1.8
- net at U2.3 (PL): now also U1.11; no longer U1.3
- net at C2.1, R2.2: now also U1.12; no longer U1.1
- net at C1.1, R1.1: now also U1.13, U1.9; no longer U1.2, U1.5
- net at R2.1: now also U1.10; no longer U1.4
- new net: U1.3, U1.5
Changed lines of the file:
@@
 $Comp
 L 7402 U1
-U 4 1 58C07186
+U 2 1 58C07186
 P 9200 6050
 F 0 "U1" H 9200 6100 50  0000 C CNN
@@
 F 2 "" H 9200 6050 50  0000 C CNN
 F 3 "" H 9200 6050 50  0000 C CNN
-	4    9200 6050
+	2    9200 6050
 	1    0    0    -1
 $EndComp
 $Comp
 L 7402 U1
-U 3 1 58C03FD3
+U 1 1 58C03FD3
 P 7550 6150
 F 0 "U1" H 7550 6200 50  0000 C CNN
@@
 F 2 "" H 7550 6150 50  0000 C CNN
 F 3 "" H 7550 6150 50  0000 C CNN
-	3    7550 6150
+	1    7550 6150
 	1    0    0    -1
 $EndComp
 $Comp
 L 7402 U1
-U 2 1 58C07EDD
+U 3 1 58C07EDD
 P 4700 5800
 F 0 "U1" H 4700 5850 50  0000 C CNN
@@
 F 2 "" H 4700 5800 50  0000 C CNN
 F 3 "" H 4700 5800 50  0000 C CNN
-	2    4700 5800
+	3    4700 5800
 	-1   0    0    1
 $EndComp
@@
 Connection ~ 4950 1800
 Wire Wire Line
-	4950 1650 4950 2100
+	4950 1650 4950 1800
+Wire Wire Line
+	4950 1800 4950 1950
+Wire Wire Line
+	4950 1950 4950 2100
 Connection ~ 4400 2100
 Wire Wire Line
@@
 	4650 1950 4300 1950
 Wire Wire Line
-	4400 1550 4400 3200
-Wire Wire Line
-	4300 1550 4300 3200
+	4400 1550 4400 2100
+Wire Wire Line
+	4400 2100 4400 3200
+Wire Wire Line
+	4300 1550 4300 1950
+Wire Wire Line
+	4300 1950 4300 3200
 Connection ~ 4200 1800
 Wire Wire Line
@@
 	4650 1650 4100 1650
 Wire Wire Line
-	4100 950  4400 950
+	4100 950  4200 950
+Wire Wire Line
+	4200 950  4250 950
+Wire Wire Line
+	4250 950  4300 950
+Wire Wire Line
+	4300 950  4400 950
 Connection ~ 4250 950
 Wire Wire Line
@@
 	5550 5650 5550 5650
 Wire Wire Line
-	3400 5350 5700 5350
+	3400 5350 5300 5350
+Wire Wire Line
+	5300 5350 5550 5350
+Wire Wire Line
+	5550 5350 5700 5350
 Wire Wire Line
 	3400 5350 3400 5600
@@
 	3500 5800 3500 5950
 Wire Wire Line
-	3400 5800 3650 5800
+	3400 5800 3500 5800
+Wire Wire Line
+	3500 5800 3650 5800
 Wire Wire Line
 	3950 5800 4100 5800
@@
 Connection ~ 8600 2900
 Wire Wire Line
-	8600 2700 8600 5950
+	8600 2700 8600 2900
+Wire Wire Line
+	8600 2900 8600 5350
+Wire Wire Line
+	8600 5350 8600 5950
 Wire Wire Line
 	8150 2900 8600 2900
@@
 Connection ~ 7100 4100
 Wire Wire Line
-	7100 4050 7100 4200
+	7100 4050 7100 4100
+Wire Wire Line
+	7100 4100 7100 4200
 Wire Wire Line
 	7300 4100 7100 4100
@@
 	7100 3000 7150 3000
 Wire Wire Line
-	7100 2500 7100 3650
+	7100 2500 7100 2700
+Wire Wire Line
+	7100 2700 7100 3000
+Wire Wire Line
+	7100 3000 7100 3600
+Wire Wire Line
+	7100 3600 7100 3650
 Wire Wire Line
 	3350 3750 3350 2900
@@
 	6700 3850 6800 3850
 Wire Wire Line
-	1650 2900 7150 2900
+	1650 2900 3350 2900
+Wire Wire Line
+	3350 2900 6700 2900
+Wire Wire Line
+	6700 2900 7150 2900
 Wire Wire Line
 	6700 2900 6700 3850
@@
 	3950 4350 3350 4350
 Wire Wire Line
-	3350 4000 3350 4500
+	3350 4000 3350 4350
+Wire Wire Line
+	3350 4350 3350 4500
 Wire Wire Line
 	3450 4000 3350 4000
@@
 	3150 4100 3450 4100
 Wire Wire Line
-	3150 3550 3150 4100
+	3150 3550 3150 3650
+Wire Wire Line
+	3150 3650 3150 4100
 Wire Wire Line
 	3450 3650 3150 3650
@@
 Connection ~ 4200 950
 Wire Wire Line
-	4200 1550 4200 3200
-Wire Wire Line
-	4100 1550 4100 3200
+	4200 1550 4200 1800
+Wire Wire Line
+	4200 1800 4200 3200
+Wire Wire Line
+	4100 1550 4100 1650
+Wire Wire Line
+	4100 1650 4100 3200
 Wire Wire Line
 	2050 5700 2050 2700
@@
 $Comp
 L 7402 U1
-U 1 1 58C07DEF
+U 4 1 58C07DEF
 P 2800 5700
 F 0 "U1" H 2800 5750 50  0000 C CNN
@@
 F 2 "" H 2800 5700 50  0000 C CNN
 F 3 "" H 2800 5700 50  0000 C CNN
-	1    2800 5700
+	4    2800 5700
 	-1   0    0    1
 $EndComp

Commit message: ouput driver
Parts:
- U1: symbol 7402 -> 7402-RESCUE-IRemote
Changed lines of the file:
@@
 $EndComp
 $Comp
-L 7402 U1
+L 7402-RESCUE-IRemote U1
 U 2 1 58C07186
 P 9200 6050
@@
 $EndComp
 $Comp
-L 7402 U1
+L 7402-RESCUE-IRemote U1
 U 1 1 58C03FD3
 P 7550 6150
@@
 $EndComp
 $Comp
-L 7402 U1
+L 7402-RESCUE-IRemote U1
 U 3 1 58C07EDD
 P 4700 5800
@@
 falling edge detector
 $Comp
-L 7402 U1
+L 7402-RESCUE-IRemote U1
 U 4 1 58C07DEF
 P 2800 5700
