File: schema/signal_generator.sch (KiCad schematic (older format))
At the start: 17 parts, among them U10 HEF4526B, U5 TLC555, U6 TLC555, U9 7402

Commit message: Schematic done
Parts:
- removed Rbl, Rpl: R, symbol R
- added C17, C18, C19: 100nF, symbol C
- R23: renamed from Rpb; value R -> 1.5k
- renumbered Cp to C16, Rba to R13, Rbb to R19, Rpa to R20
Connections:
- wire segments 84 -> 81
Other:
- note added: "Downcounter"
- note removed: "Decounter"
- moved on the sheet: U6
Changed lines of the file:
@@
 encoding utf-8
 Sheet 6 6
-Title ""
+Title "Signal Generator"
 Date ""
 Rev ""
@@
 $EndComp
 $Comp
-L +BATT #PWR49
+L +BATT #PWR66
 U 1 1 5912CCA8
 P 6750 1050
-F 0 "#PWR49" H 6750 900 50  0001 C CNN
+F 0 "#PWR66" H 6750 900 50  0001 C CNN
 F 1 "+BATT" H 6750 1190 50  0000 C CNN
 F 2 "" H 6750 1050 50  0000 C CNN
@@
 $EndComp
 $Comp
-L GND #PWR50
+L GND #PWR67
 U 1 1 5912ED7F
 P 7600 3000
-F 0 "#PWR50" H 7600 2750 50  0001 C CNN
+F 0 "#PWR67" H 7600 2750 50  0001 C CNN
 F 1 "GND" H 7600 2850 50  0000 C CNN
 F 2 "" H 7600 3000 50  0000 C CNN
@@
 $EndComp
 $Comp
-L GND #PWR48
+L GND #PWR65
 U 1 1 59130203
 P 6450 4700
-F 0 "#PWR48" H 6450 4450 50  0001 C CNN
+F 0 "#PWR65" H 6450 4450 50  0001 C CNN
 F 1 "GND" H 6450 4550 50  0000 C CNN
 F 2 "" H 6450 4700 50  0000 C CNN
@@
 $EndComp
 $Comp
-L +BATT #PWR46
+L +BATT #PWR63
 U 1 1 591303F3
 P 6250 3250
-F 0 "#PWR46" H 6250 3100 50  0001 C CNN
+F 0 "#PWR63" H 6250 3100 50  0001 C CNN
 F 1 "+BATT" H 6250 3390 50  0000 C CNN
 F 2 "" H 6250 3250 50  0000 C CNN
@@
 $EndComp
 $Comp
-L +BATT #PWR41
+L +BATT #PWR53
 U 1 1 591329F1
 P 2000 1950
-F 0 "#PWR41" H 2000 1800 50  0001 C CNN
+F 0 "#PWR53" H 2000 1800 50  0001 C CNN
 F 1 "+BATT" H 2000 2090 50  0000 C CNN
 F 2 "" H 2000 1950 50  0000 C CNN
@@
 $EndComp
 $Comp
-L R Rbb
+L R R19
 U 1 1 59132C26
 P 1050 3000
-F 0 "Rbb" V 1130 3000 50  0000 C CNN
+F 0 "R19" V 1130 3000 50  0000 C CNN
 F 1 "467k" V 1050 3000 50  0000 C CNN
 F 2 "" V 980 3000 50  0000 C CNN
@@
 $EndComp
 $Comp
-L R Rbl
-U 1 1 59132D4D
-P 2950 2450
-F 0 "Rbl" V 3030 2450 50  0000 C CNN
-F 1 "R" V 2950 2450 50  0000 C CNN
-F 2 "" V 2880 2450 50  0000 C CNN
-F 3 "" H 2950 2450 50  0000 C CNN
-	1    2950 2450
-	1    0    0    -1
-$EndComp
-$Comp
-L GND #PWR42
+L GND #PWR54
 U 1 1 59132E59
 P 2000 3700
-F 0 "#PWR42" H 2000 3450 50  0001 C CNN
+F 0 "#PWR54" H 2000 3450 50  0001 C CNN
 F 1 "GND" H 2000 3550 50  0000 C CNN
 F 2 "" H 2000 3700 50  0000 C CNN
@@
 NoConn ~ 2500 3050
 $Comp
-L R Rba
+L R R13
 U 1 1 59133297
 P 1050 2500
-F 0 "Rba" V 1130 2500 50  0000 C CNN
+F 0 "R13" V 1130 2500 50  0000 C CNN
 F 1 "556k" V 1050 2500 50  0000 C CNN
 F 2 "" V 980 2500 50  0000 C CNN
@@
 Burst timer (th = 70ms, tl = 30ms)
 Text Notes 5450 2050 0    60   ~ 0
-Decounter
+Downcounter
 $Comp
 L TLC555 U6
 U 1 1 5913C644
-P 2000 5850
-F 0 "U6" H 1900 6275 50  0000 R CNN
-F 1 "TLC555" H 1900 6200 50  0000 R CNN
-F 2 "" H 2050 5600 50  0000 L CNN
-F 3 "" H 2650 5300 50  0000 C CNN
-	1    2000 5850
-	1    0    0    -1
-$EndComp
-$Comp
-L +BATT #PWR43
+P 2000 5900
+F 0 "U6" H 1900 6325 50  0000 R CNN
+F 1 "TLC555" H 1900 6250 50  0000 R CNN
+F 2 "" H 2050 5650 50  0000 L CNN
+F 3 "" H 2650 5350 50  0000 C CNN
+	1    2000 5900
+	1    0    0    -1
+$EndComp
+$Comp
+L +BATT #PWR55
 U 1 1 5913C64A
 P 2000 4850
-F 0 "#PWR43" H 2000 4700 50  0001 C CNN
+F 0 "#PWR55" H 2000 4700 50  0001 C CNN
 F 1 "+BATT" H 2000 4990 50  0000 C CNN
 F 2 "" H 2000 4850 50  0000 C CNN
@@
 $EndComp
 $Comp
-L R Rpb
+L R R23
 U 1 1 5913C657
 P 1050 5900
-F 0 "Rpb" V 1130 5900 50  0000 C CNN
-F 1 "R" V 1050 5900 50  0000 C CNN
+F 0 "R23" V 1130 5900 50  0000 C CNN
+F 1 "1.5k" V 1050 5900 50  0000 C CNN
 F 2 "" V 980 5900 50  0000 C CNN
 F 3 "" H 1050 5900 50  0000 C CNN
@@
 $EndComp
 $Comp
-L R Rpl
-U 1 1 5913C665
-P 2950 5350
-F 0 "Rpl" V 3030 5350 50  0000 C CNN
-F 1 "R" V 2950 5350 50  0000 C CNN
-F 2 "" V 2880 5350 50  0000 C CNN
-F 3 "" H 2950 5350 50  0000 C CNN
-	1    2950 5350
-	1    0    0    -1
-$EndComp
-$Comp
-L GND #PWR44
+L GND #PWR56
 U 1 1 5913C66F
 P 2000 6600
-F 0 "#PWR44" H 2000 6350 50  0001 C CNN
+F 0 "#PWR56" H 2000 6350 50  0001 C CNN
 F 1 "GND" H 2000 6450 50  0000 C CNN
 F 2 "" H 2000 6600 50  0000 C CNN
@@
 NoConn ~ 2500 5950
 $Comp
-L R Rpa
+L R R20
 U 1 1 5913C678
 P 1050 5400
-F 0 "Rpa" V 1130 5400 50  0000 C CNN
+F 0 "R20" V 1130 5400 50  0000 C CNN
 F 1 "12k" V 1050 5400 50  0000 C CNN
 F 2 "" V 980 5400 50  0000 C CNN
@@
 $EndComp
 $Comp
-L C Cp
+L C C16
 U 1 1 5913C686
 P 1450 6350
-F 0 "Cp" H 1475 6450 50  0000 L CNN
+F 0 "C16" H 1475 6450 50  0000 L CNN
 F 1 "100nF" H 1475 6250 50  0000 L CNN
 F 2 "" H 1488 6200 50  0000 C CNN
@@
 $EndComp
 $Comp
-L GND #PWR45
+L GND #PWR62
 U 1 1 591D7268
 P 5950 5750
-F 0 "#PWR45" H 5950 5500 50  0001 C CNN
+F 0 "#PWR62" H 5950 5500 50  0001 C CNN
 F 1 "GND" H 5950 5600 50  0000 C CNN
 F 2 "" H 5950 5750 50  0000 C CNN
@@
 	6450 2950 6450 3300
 Wire Wire Line
-	2500 2950 6450 2950
-Wire Wire Line
 	5950 4100 5650 4100
 Wire Wire Line
@@
 	2500 2750 2700 2750
 Wire Wire Line
-	2700 2100 2700 2750
-Wire Wire Line
-	1050 2100 2950 2100
+	2700 2750 2700 2100
 Connection ~ 2000 2100
-Wire Wire Line
-	2950 2100 2950 2300
-Connection ~ 2700 2100
-Wire Wire Line
-	2950 2950 2950 2600
-Connection ~ 2950 2950
 Wire Wire Line
 	2000 3250 2000 3700
@@
 	2500 5650 2700 5650
 Wire Wire Line
-	1050 5000 2950 5000
+	1050 5000 2600 5000
 Connection ~ 2000 5000
 Wire Wire Line
 	2500 5850 4350 5850
-Wire Wire Line
-	2950 5000 2950 5200
-Wire Wire Line
-	2950 5500 2950 5850
-Connection ~ 2950 5850
 Wire Wire Line
 	2000 6150 2000 6600
@@
 Connection ~ 7900 5300
 $Comp
-L GND #PWR47
+L GND #PWR64
 U 1 1 591DA0C5
 P 6300 6700
-F 0 "#PWR47" H 6300 6450 50  0001 C CNN
+F 0 "#PWR64" H 6300 6450 50  0001 C CNN
 F 1 "GND" H 6300 6550 50  0000 C CNN
 F 2 "" H 6300 6700 50  0000 C CNN
@@
 	9400 5400 10100 5400
 $Comp
-L +BATT #PWR?
+L +BATT #PWR59
 U 1 1 593EF96A
 P 5600 3350
-F 0 "#PWR?" H 5600 3200 50  0001 C CNN
+F 0 "#PWR59" H 5600 3200 50  0001 C CNN
 F 1 "+BATT" H 5600 3490 50  0000 C CNN
 F 2 "" H 5600 3350 50  0000 C CNN
@@
 	4600 3850 5950 3850
 Connection ~ 4600 5500
+$Comp
+L C C19
+U 1 1 593EC8C9
+P 5700 2450
+F 0 "C19" H 5725 2550 50  0000 L CNN
+F 1 "100nF" H 5725 2350 50  0000 L CNN
+F 2 "" H 5738 2300 50  0000 C CNN
+F 3 "" H 5700 2450 50  0000 C CNN
+	1    5700 2450
+	1    0    0    -1
+$EndComp
+$Comp
+L GND #PWR61
+U 1 1 593EC93C
+P 5700 2600
+F 0 "#PWR61" H 5700 2350 50  0001 C CNN
+F 1 "GND" H 5700 2450 50  0000 C CNN
+F 2 "" H 5700 2600 50  0000 C CNN
+F 3 "" H 5700 2600 50  0000 C CNN
+	1    5700 2600
+	1    0    0    -1
+$EndComp
+$Comp
+L +BATT #PWR60
+U 1 1 593EC99B
+P 5700 2300
+F 0 "#PWR60" H 5700 2150 50  0001 C CNN
+F 1 "+BATT" H 5700 2440 50  0000 C CNN
+F 2 "" H 5700 2300 50  0000 C CNN
+F 3 "" H 5700 2300 50  0000 C CNN
+	1    5700 2300
+	1    0    0    -1
+$EndComp
+Wire Wire Line
+	2500 2950 6450 2950
+$Comp
+L C C17
+U 1 1 593ED55F
+P 2300 2300
+F 0 "C17" H 2325 2400 50  0000 L CNN
+F 1 "100nF" H 2325 2200 50  0000 L CNN
+F 2 "" H 2338 2150 50  0000 C CNN
+F 3 "" H 2300 2300 50  0000 C CNN
+	1    2300 2300
+	1    0    0    -1
+$EndComp
+$Comp
+L GND #PWR57
+U 1 1 593ED565
+P 2300 2450
+F 0 "#PWR57" H 2300 2200 50  0001 C CNN
+F 1 "GND" H 2300 2300 50  0000 C CNN
+F 2 "" H 2300 2450 50  0000 C CNN
+F 3 "" H 2300 2450 50  0000 C CNN
+	1    2300 2450
+	1    0    0    -1
+$EndComp
+$Comp
+L C C18
+U 1 1 593ED594
+P 2600 5150
+F 0 "C18" H 2625 5250 50  0000 L CNN
+F 1 "100nF" H 2625 5050 50  0000 L CNN
+F 2 "" H 2638 5000 50  0000 C CNN
+F 3 "" H 2600 5150 50  0000 C CNN
+	1    2600 5150
+	1    0    0    -1
+$EndComp
+$Comp
+L GND #PWR58
+U 1 1 593ED59A
+P 2600 5300
+F 0 "#PWR58" H 2600 5050 50  0001 C CNN
+F 1 "GND" H 2600 5150 50  0000 C CNN
+F 2 "" H 2600 5300 50  0000 C CNN
+F 3 "" H 2600 5300 50  0000 C CNN
+	1    2600 5300
+	1    0    0    -1
+$EndComp
+Wire Wire Line
+	2700 2100 1050 2100
+Connection ~ 2300 2100
+Wire Wire Line
+	2300 2150 2300 2100
 $EndSCHEMATC
