File: schema/recevier_filter.sch (KiCad schematic (older format))
At the start: 15 parts, among them U7 LMC6482, U8 LM393

Commit message: Add missing decoupling capacitors
Parts:
- added C23: 100nF, symbol C
Connections:
- net +5V: now also C23.1
- net GND: now also C23.2
Changed lines of the file:
@@
 $EndComp
 $Comp
-L GND #PWR12
+L GND #PWR14
 U 1 1 59106802
 P 4750 3950
-F 0 "#PWR12" H 4750 3700 50  0001 C CNN
+F 0 "#PWR14" H 4750 3700 50  0001 C CNN
 F 1 "GND" H 4750 3800 50  0000 C CNN
 F 2 "" H 4750 3950 50  0000 C CNN
@@
 $EndComp
 Wire Wire Line
-	3300 3650 3450 3650
-Wire Wire Line
-	3450 3650 4300 3650
-Wire Wire Line
-	4600 3650 4750 3650
-Wire Wire Line
-	4750 3650 5150 3650
+	3300 3650 4300 3650
+Wire Wire Line
+	4600 3650 5150 3650
 Connection ~ 4750 3650
 $Comp
@@
 $EndComp
 Wire Wire Line
-	1700 3750 2450 3750
-Wire Wire Line
-	2450 3750 2700 3750
+	1700 3750 2700 3750
 Wire Wire Line
 	1250 3750 1250 3950
@@
 $EndComp
 Wire Wire Line
-	6200 3550 6250 3550
-Wire Wire Line
-	6250 3550 8100 3550
-Wire Wire Line
-	5400 4200 5500 4200
-Wire Wire Line
-	5500 4200 5650 4200
+	6200 3550 8100 3550
+Wire Wire Line
+	5400 4200 5650 4200
 Connection ~ 5500 4200
 Wire Wire Line
@@
 Connection ~ 6250 3550
 $Comp
-L GND #PWR13
+L GND #PWR15
 U 1 1 5910AC6D
 P 5000 4200
-F 0 "#PWR13" H 5000 3950 50  0001 C CNN
+F 0 "#PWR15" H 5000 3950 50  0001 C CNN
 F 1 "GND" H 5000 4050 50  0000 C CNN
 F 2 "" H 5000 4200 50  0000 C CNN
@@
 	5000 4200 5100 4200
 $Comp
-L +5V #PWR14
+L +5V #PWR16
 U 1 1 5910ADF1
 P 5800 3250
-F 0 "#PWR14" H 5800 3100 50  0001 C CNN
+F 0 "#PWR16" H 5800 3100 50  0001 C CNN
 F 1 "+5V" H 5800 3390 50  0000 C CNN
 F 2 "" H 5800 3250 50  0000 C CNN
@@
 $EndComp
 $Comp
-L GND #PWR15
+L GND #PWR17
 U 1 1 5910B09A
 P 5800 3850
-F 0 "#PWR15" H 5800 3600 50  0001 C CNN
+F 0 "#PWR17" H 5800 3600 50  0001 C CNN
 F 1 "GND" H 5800 3700 50  0000 C CNN
 F 2 "" H 5800 3850 50  0000 C CNN
@@
 Connection ~ 2450 3750
 Wire Wire Line
-	2450 2650 2450 2950
-Wire Wire Line
-	2450 2950 2450 3750
-Wire Wire Line
-	3450 2650 3450 2950
-Wire Wire Line
-	3450 2950 3450 3650
+	2450 2650 2450 3750
+Wire Wire Line
+	3450 2650 3450 3650
 $Comp
 L C C8
@@
 $EndComp
 $Comp
-L GND #PWR17
+L GND #PWR19
 U 1 1 5924CCA3
 P 7600 4250
-F 0 "#PWR17" H 7600 4000 50  0001 C CNN
+F 0 "#PWR19" H 7600 4000 50  0001 C CNN
 F 1 "GND" H 7600 4100 50  0000 C CNN
 F 2 "" H 7600 4250 50  0000 C CNN
@@
 $EndComp
 $Comp
-L GND #PWR20
+L GND #PWR22
 U 1 1 5924CE19
 P 8300 4000
-F 0 "#PWR20" H 8300 3750 50  0001 C CNN
+F 0 "#PWR22" H 8300 3750 50  0001 C CNN
 F 1 "GND" H 8300 3850 50  0000 C CNN
 F 2 "" H 8300 4000 50  0000 C CNN
@@
 $EndComp
 $Comp
-L +5V #PWR19
+L +5V #PWR21
 U 1 1 5924CE97
 P 8300 2650
-F 0 "#PWR19" H 8300 2500 50  0001 C CNN
+F 0 "#PWR21" H 8300 2500 50  0001 C CNN
 F 1 "+5V" H 8300 2790 50  0000 C CNN
 F 2 "" H 8300 2650 50  0000 C CNN
@@
 $EndComp
 $Comp
-L +5V #PWR16
+L +5V #PWR18
 U 1 1 5924CFDF
 P 7600 2750
-F 0 "#PWR16" H 7600 2600 50  0001 C CNN
+F 0 "#PWR18" H 7600 2600 50  0001 C CNN
 F 1 "+5V" H 7600 2890 50  0000 C CNN
 F 2 "" H 7600 2750 50  0000 C CNN
@@
 $EndComp
 $Comp
-L +5V #PWR21
+L +5V #PWR23
 U 1 1 5924DE3C
 P 8900 2950
-F 0 "#PWR21" H 8900 2800 50  0001 C CNN
+F 0 "#PWR23" H 8900 2800 50  0001 C CNN
 F 1 "+5V" H 8900 3090 50  0000 C CNN
 F 2 "" H 8900 2950 50  0000 C CNN
@@
 $EndComp
 $Comp
-L GND #PWR18
+L GND #PWR20
 U 1 1 5925407F
 P 7950 2950
-F 0 "#PWR18" H 7950 2700 50  0001 C CNN
+F 0 "#PWR20" H 7950 2700 50  0001 C CNN
 F 1 "GND" H 7950 2800 50  0000 C CNN
 F 2 "" H 7950 2950 50  0000 C CNN
@@
 $EndComp
 Wire Wire Line
-	8700 3450 8900 3450
-Wire Wire Line
-	8900 3450 9700 3450
-Wire Wire Line
-	8900 3300 8900 3450
-Wire Wire Line
-	8900 3450 8900 3800
+	8700 3450 9700 3450
+Wire Wire Line
+	8900 3300 8900 3800
 Connection ~ 8900 3450
 Wire Wire Line
 	7600 2750 7600 2900
 Wire Wire Line
-	7600 3200 7600 3350
-Wire Wire Line
-	7600 3350 7600 3800
-Wire Wire Line
-	7600 3800 7600 3850
+	7600 3200 7600 3850
 Wire Wire Line
 	7600 3350 8100 3350
@@
 $EndComp
 $Comp
-L GND #PWR11
+L GND #PWR13
 U 1 1 593EB2BE
 P 4450 3000
-F 0 "#PWR11" H 4450 2750 50  0001 C CNN
+F 0 "#PWR13" H 4450 2750 50  0001 C CNN
 F 1 "GND" H 4450 2850 50  0000 C CNN
 F 2 "" H 4450 3000 50  0000 C CNN
@@
 $EndComp
 $Comp
-L +5V #PWR10
+L +5V #PWR12
 U 1 1 593EB309
 P 4450 2700
-F 0 "#PWR10" H 4450 2550 50  0001 C CNN
+F 0 "#PWR12" H 4450 2550 50  0001 C CNN
 F 1 "+5V" H 4450 2840 50  0000 C CNN
 F 2 "" H 4450 2700 50  0000 C CNN
@@
 	1    0    0    -1
 $EndComp
+$Comp
+L C C23
+U 1 1 593ED0F2
+P 3750 2850
+F 0 "C23" H 3775 2950 50  0000 L CNN
+F 1 "100nF" H 3775 2750 50  0000 L CNN
+F 2 "" H 3788 2700 50  0000 C CNN
+F 3 "" H 3750 2850 50  0000 C CNN
+	1    3750 2850
+	1    0    0    -1
+$EndComp
+$Comp
+L GND #PWR11
+U 1 1 593ED0F8
+P 3750 3000
+F 0 "#PWR11" H 3750 2750 50  0001 C CNN
+F 1 "GND" H 3750 2850 50  0000 C CNN
+F 2 "" H 3750 3000 50  0000 C CNN
+F 3 "" H 3750 3000 50  0000 C CNN
+	1    3750 3000
+	1    0    0    -1
+$EndComp
+$Comp
+L +5V #PWR10
+U 1 1 593ED0FE
+P 3750 2700
+F 0 "#PWR10" H 3750 2550 50  0001 C CNN
+F 1 "+5V" H 3750 2840 50  0000 C CNN
+F 2 "" H 3750 2700 50  0000 C CNN
+F 3 "" H 3750 2700 50  0000 C CNN
+	1    3750 2700
+	1    0    0    -1
+$EndComp
